File: peltier_driver_pcb/Arduino_Nano_shield/Arduino_Nano_shield.kicad_pcb (KiCad board)
At the start: 2 copper layers, 61 x 51 mm, 7 parts, among them J1 Conn_02x10_Top_Bottom, J2 Conn_02x10_Top_Bottom

Commit message: final touches for second design iteration
Parts:
- moved H1 2.03 mm to (149.9, 93.3)
- moved H4 2.00 mm to (96.5, 93.3)
- moved XA2 2.00 mm to (143.5, 86.3)
Routing:
- net +3V3: track 50.5 -> 54.1 mm
- net PWM1: track 37.9 -> 40.1 mm
- net PWM3: track 38.2 -> 40.2 mm
- net SDA: track 31.5 -> 33.5 mm
- net T_sense2: track 34.4 -> 36.4 mm
- net T_sense1: track 30.9 -> 32.9 mm
- net SCL: track 27.9 -> 29.9 mm
- net PWM5: track 30.6 -> 32.6 mm
- net PWM4: track 34.6 -> 36.6 mm
- net PWM0: track 35.4 -> 37.4 mm
- net I_sense_2: track 39.5 -> 41.5 mm
- net I_sense_1: track 34.4 -> 36.4 mm
- net D8: track 42.0 -> 44.0 mm
- net D2: track 37.0 -> 39.0 mm
- net D13: track 9.90 -> 11.9 mm
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Other:
- board size 61 x 51 mm -> 61.3 x 54 mm
